Commit message: remove: ToF (VL53L5CX) dropped — LiDAR covers all obstacle detection

File: ros2_ws/src/amr_description/urdf/sensors.urdf.xacro (robot description, xacro)
@@ -19,11 +19,4 @@
     <child  link="imu_link"/>
     <origin xyz="0.0 0.0 0.020" rpy="0 0 0"/>  <!-- UPDATE with measured offset -->
-  </joint>
-  <!-- ToF sensor — forward-facing at front of robot -->
-  <link name="tof_link"/>
-  <joint name="tof_joint" type="fixed">
-    <parent link="base_link"/>
-    <child  link="tof_link"/>
-    <origin xyz="0.370 0.0 0.080" rpy="0 0 0"/>  <!-- UPDATE with measured offset -->
   </joint>
   <!-- Gazebo sensor plugins (only active when use_sim:=true) -->

Commit message: feat: Phase 5 — amr_slam package (slam_toolbox online_async) + LiDAR TF measured

File: ros2_ws/src/amr_description/urdf/sensors.urdf.xacro (robot description, xacro)
@@ -11,5 +11,5 @@
     <parent link="base_link"/>
     <child  link="base_laser"/>
-    <origin xyz="0.0 0.0 0.080" rpy="0 0 0"/>  <!-- UPDATE with measured offset -->
+    <origin xyz="0.2995 0.0 0.13" rpy="0 0 0"/>
   </joint>
   <!-- IMU mount -->

Commit message: fix: LiDAR TF x=0.327m (center of scan disc, measured)

File: ros2_ws/src/amr_description/urdf/sensors.urdf.xacro (robot description, xacro)
@@ -11,5 +11,5 @@
     <parent link="base_link"/>
     <child  link="base_laser"/>
-    <origin xyz="0.2995 0.0 0.13" rpy="0 0 0"/>
+    <origin xyz="0.327 0.0 0.13" rpy="0 0 0"/>
   </joint>
   <!-- IMU mount -->

Commit message: fix: declare 180deg LiDAR mounting yaw offset in URDF
User reported scan detections mirrored front<->back AND left<->right --
a person standing in front of the robot showed up "behind" it in RViz.
That combined swap is the signature of a 180 deg yaw mounting offset, not
a simple flip: the LiDAR's physical zero-angle reference points toward the
robot's rear, but base_laser_joint declared rpy="0 0 0" (zero pointing
forward). Setting yaw=pi tells TF the true mounting orientation so scan
ranges land in their correct real-world positions relative to base_link.

File: ros2_ws/src/amr_description/urdf/sensors.urdf.xacro (robot description, xacro)
@@ -11,5 +11,11 @@
     <parent link="base_link"/>
     <child  link="base_laser"/>
-    <origin xyz="0.327 0.0 0.13" rpy="0 0 0"/>
+    <!-- yaw = pi: LiDAR is physically mounted rotated 180 deg from base_link's
+         forward axis -- its own zero-angle reference points toward the robot's
+         REAR. Without this offset, TF reports scan detections mirrored front<->
+         back AND left<->right (a person standing in front of the robot showed
+         up "behind" it in RViz, and vice versa -- the signature of a missing
+         180 deg yaw declaration, not a left/right flip). -->
+    <origin xyz="0.327 0.0 0.13" rpy="0 0 ${pi}"/>
   </joint>
   <!-- IMU mount -->
