Commit message: fix: correct chassis dimensions to 71.5×56.5 cm (measured), update inertia

File: ros2_ws/src/amr_description/urdf/amr.urdf.xacro (robot description, xacro)
@@ -4,5 +4,5 @@
   <xacro:include filename="$(find amr_description)/urdf/wheels.urdf.xacro"/>
   <xacro:include filename="$(find amr_description)/urdf/sensors.urdf.xacro"/>
-  <!-- Robot dimensions: 75cm long, 58.5cm wide -->
+  <!-- Robot dimensions: 71.5cm long, 56.5cm wide (measured) -->
   <!-- MEASURE lx (half-wheelbase) and ly (half-track) from physical frame -->
   <xacro:property name="lx" value="0.275"/>  <!-- half front-to-rear axle distance — UPDATE -->
@@ -19,13 +19,14 @@
   <link name="base_link">
     <visual>
-      <geometry><box size="0.750 0.585 0.060"/></geometry>
+      <geometry><box size="0.715 0.565 0.060"/></geometry>
       <material name="grey"><color rgba="0.6 0.6 0.6 1"/></material>
     </visual>
     <collision>
-      <geometry><box size="0.750 0.585 0.060"/></geometry>
+      <geometry><box size="0.715 0.565 0.060"/></geometry>
     </collision>
     <inertial>
       <mass value="8.000"/>
-      <inertia ixx="0.2282" iyy="0.3750" izz="0.5844"
+      <!-- ixx=(1/12)*8*(0.565²+0.060²), iyy=(1/12)*8*(0.715²+0.060²), izz=(1/12)*8*(0.715²+0.565²) -->
+      <inertia ixx="0.2152" iyy="0.3432" izz="0.5537"
                ixy="0" ixz="0" iyz="0"/>
     </inertial>

Commit message: feat: Phase 6 — Nav2 navigation (SmacPlannerLattice + MPPI Omni + collision_monitor)
- amr_nav package: nav2_params.yaml (behavior_server/Jazzy, no ToF, CostCritic),
  collision_monitor.yaml (/scan only), nav2.launch.py (OpaqueFunction injects
  lattice_filepath at launch time — avoids lifecycle race condition)
- OMNI lattice primitives: 5cm grid, 16 headings, 144 trajectories (official
  Nav2 sample, no standalone generator binary in this Humble install)
- amr.launch.py: replace twist_to_reference bridge with topic_tools relay
  /cmd_vel_safe → /mecanum_drive_controller/reference (Nav2 chain:
  MPPI→/cmd_vel→collision_monitor→/cmd_vel_safe→relay→controller)
- controllers.yaml: wheel kinematics locked (sum=0.486: lx=0.231+ly=0.255)
- URDF: lx=0.231m, ly=0.255m (measured from physical robot 2026-05-31)

File: ros2_ws/src/amr_description/urdf/amr.urdf.xacro (robot description, xacro)
@@ -6,6 +6,6 @@
   <!-- Robot dimensions: 71.5cm long, 56.5cm wide (measured) -->
   <!-- MEASURE lx (half-wheelbase) and ly (half-track) from physical frame -->
-  <xacro:property name="lx" value="0.275"/>  <!-- half front-to-rear axle distance — UPDATE -->
-  <xacro:property name="ly" value="0.220"/>  <!-- half left-to-right axle distance — UPDATE -->
+  <xacro:property name="lx" value="0.231"/>  <!-- half front-to-rear axle distance: 46.2cm/2 (measured) -->
+  <xacro:property name="ly" value="0.255"/>  <!-- half left-to-right axle distance: 51.0cm/2 (measured) -->
   <xacro:property name="wheel_z" value="-0.060"/>  <!-- wheel centre height from base_link -->
   <!-- Base footprint -->

Commit message: feat(description): visual upgrade — charcoal chassis, blue accent, orange wheels, LEDs, sensor tower

File: ros2_ws/src/amr_description/urdf/amr.urdf.xacro (robot description, xacro)
@@ -18,7 +18,14 @@
   <!-- Main chassis -->
   <link name="base_link">
-    <visual>
+    <!-- Charcoal body -->
+    <visual name="chassis_body">
       <geometry><box size="0.715 0.565 0.060"/></geometry>
-      <material name="grey"><color rgba="0.6 0.6 0.6 1"/></material>
+      <material name="charcoal"><color rgba="0.15 0.15 0.18 1"/></material>
+    </visual>
+    <!-- Bright blue perimeter accent strip -->
+    <visual name="chassis_accent">
+      <origin xyz="0 0 0.032" rpy="0 0 0"/>
+      <geometry><box size="0.720 0.570 0.004"/></geometry>
+      <material name="blue_accent"><color rgba="0.2 0.5 1.0 1"/></material>
     </visual>
     <collision>
@@ -37,4 +44,34 @@
   <xacro:mecanum_wheel name="wheel_RL" x="-${lx}" y=" ${ly}" z="${wheel_z}" reflect_y="1"/>
   <xacro:mecanum_wheel name="wheel_RR" x="-${lx}" y="-${ly}" z="${wheel_z}" reflect_y="-1"/>
+  <!-- Sensor tower — matte black cylinder stack below LiDAR -->
+  <link name="sensor_tower">
+    <visual>
+      <geometry><cylinder radius="0.042" length="0.065"/></geometry>
+      <material name="matte_black"><color rgba="0.08 0.08 0.08 1"/></material>
+    </visual>
+  </link>
+  <joint name="sensor_tower_joint" type="fixed">
+    <parent link="base_link"/>
+    <child  link="sensor_tower"/>
+    <origin xyz="0.327 0.0 0.063" rpy="0 0 0"/>
+  </joint>
+  <!-- Corner LED indicator spheres -->
+  <xacro:macro name="corner_led" params="name x y">
+    <link name="${name}">
+      <visual>
+        <geometry><sphere radius="0.013"/></geometry>
+        <material name="led_green"><color rgba="0.1 0.9 0.3 1"/></material>
+      </visual>
+    </link>
+    <joint name="${name}_joint" type="fixed">
+      <parent link="base_link"/>
+      <child  link="${name}"/>
+      <origin xyz="${x} ${y} 0.032" rpy="0 0 0"/>
+    </joint>
+  </xacro:macro>
+  <xacro:corner_led name="led_FL" x=" 0.340" y=" 0.265"/>
+  <xacro:corner_led name="led_FR" x=" 0.340" y="-0.265"/>
+  <xacro:corner_led name="led_RL" x="-0.340" y=" 0.265"/>
+  <xacro:corner_led name="led_RR" x="-0.340" y="-0.265"/>
   <!-- ros2_control hardware interface — switches between sim and real -->
   <ros2_control name="AMRSystem" type="system">

File: ros2_ws/src/amr_description/urdf/sensors.urdf.xacro (robot description, xacro)
@@ -46,5 +46,5 @@
         </lidar>
         <always_on>true</always_on>
-        <visualize>false</visualize>
+        <visualize>true</visualize>
       </sensor>
     </gazebo>

File: ros2_ws/src/amr_description/urdf/wheels.urdf.xacro (robot description, xacro)
@@ -6,5 +6,5 @@
         <geometry><cylinder length="0.04" radius="0.030"/></geometry>
         <origin xyz="0 0 0" rpy="${pi/2} 0 0"/>
-        <material name="black"><color rgba="0.1 0.1 0.1 1"/></material>
+        <material name="orange_wheel"><color rgba="0.95 0.55 0.1 1"/></material>
       </visual>
       <collision>
